File: Adafruit Sparkle Motion WLED Friend.brd (EAGLE design)
At the start: 50.8 x 33.1 mm, 66 parts, among them IC1 CH343P, IC2 ICS-43434, IC4 74LVC2G34GW, IC5 74LVC2G34GW, Q1 AONR21307, Q5 DUAL NPN, SW1 KMR2, SW2 KMR2, SW3 SWITCH_SP3T_SMD_MSK13C01, U2 NCP718ASN500T1G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

Commit message: shop image & final board silk
Parts:
- added PLABEL0: (no value), pinguin:PLABEL0
- added PLABEL1: (no value), pinguin:PLABEL1
- added PLABEL10: (no value), pinguin:PLABEL10
- added PLABEL11: (no value), pinguin:PLABEL11
- added PLABEL13: (no value), pinguin:PLABEL13
- added PLABEL14: (no value), pinguin:PLABEL14
- added PLABEL16: (no value), pinguin:PLABEL16
- added PLABEL17: (no value), pinguin:PLABEL17
- added PLABEL19: (no value), pinguin:PLABEL19
- added PLABEL2: (no value), pinguin:PLABEL2
- added PLABEL20: (no value), pinguin:PLABEL20
- added PLABEL21: (no value), pinguin:PLABEL21
- added PLABEL22: (no value), pinguin:PLABEL22
- added PLABEL23: (no value), pinguin:PLABEL23
- added PLABEL24: (no value), pinguin:PLABEL24
- added PLABEL25: (no value), pinguin:PLABEL25
- added PLABEL26: (no value), pinguin:PLABEL26
- added PLABEL27: (no value), pinguin:PLABEL27
- added PLABEL28: (no value), pinguin:PLABEL28
- added PLABEL29: (no value), pinguin:PLABEL29
- added PLABEL3: (no value), pinguin:PLABEL3
- added PLABEL30: (no value), pinguin:PLABEL30
- added PLABEL31: (no value), pinguin:PLABEL31
- added PLABEL32: (no value), pinguin:PLABEL32
- added PLABEL33: (no value), pinguin:PLABEL33
- added PLABEL34: (no value), pinguin:PLABEL34
- added PLABEL35: (no value), pinguin:PLABEL35
- added PLABEL36: (no value), pinguin:PLABEL36
- added PLABEL37: (no value), pinguin:PLABEL37
- added PLABEL38: (no value), pinguin:PLABEL38
- added PLABEL39: (no value), pinguin:PLABEL39
- added PLABEL4: (no value), pinguin:PLABEL4
- added PLABEL40: (no value), pinguin:PLABEL40
- added PLABEL41: (no value), pinguin:PLABEL41
- added PLABEL42: (no value), pinguin:PLABEL42
- added PLABEL43: (no value), pinguin:PLABEL43
- added PLABEL44: (no value), pinguin:PLABEL44
- added PLABEL45: (no value), pinguin:PLABEL45
- added PLABEL46: (no value), pinguin:PLABEL46
- added PLABEL47: (no value), pinguin:PLABEL47
- added PLABEL48: (no value), pinguin:PLABEL48
- added PLABEL49: (no value), pinguin:PLABEL49
- added PLABEL50: (no value), pinguin:PLABEL50
- added PLABEL51: (no value), pinguin:PLABEL51
- added PLABEL52: (no value), pinguin:PLABEL52
- added PLABEL53: (no value), pinguin:PLABEL53
- added PLABEL54: (no value), pinguin:PLABEL54
- added PLABEL55: (no value), pinguin:PLABEL55
- added PLABEL56: (no value), pinguin:PLABEL56
- added PLABEL6: (no value), pinguin:PLABEL6
- added PLABEL7: (no value), pinguin:PLABEL7
- added PLABEL8: (no value), pinguin:PLABEL8
- added PLABEL9: (no value), pinguin:PLABEL9
- added TP3, TP4: (no value), microbuilder:TESTPOINT_ROUND_1.5MM
- added U$46: (no value), microbuilder:ADAFRUIT_5MM
- added U$50: (no value), microbuilder:ADAFRUIT_TEXT_20MM
- R12: value 47K -> 10K
- moved TP1 0.18 mm to (41.8, 20.8)
- moved R2 0.13 mm to (9.65, 24.9)
- moved TP2 0.13 mm to (41.8, 23.5)
Connections:
- net !RESET: now also TP3.P$1
- net GPIO0: now also TP4.P$1
Routing:
- net GPIO0: track 36.9 -> 40.8 mm, vias 3 -> 4
- net !RESET: track 49.0 -> 50.6 mm, vias 3 -> 4
Other:
- board text added: "!!! WARNING !!! VERIFY DC/PD VOLTS NOT HIGHER THAN LED MAX VIN!!!"
- board text added: "#19"
- board text added: "#21"
- board text added: "#22"
- board text added: "10"
- board text added: "18"
- board text added: "19"
- board text added: "21"
- board text added: "22"
- board text added: "23"
- board text added: "3.3V"
- board text added: "5-24V"
- board text added: "5A Fuse"
- board text added: "5V Level Outputs S1:21 S2:22 S3:19 S4:23"
- board text added: "5V logic out"
- board text added: "5V~24VDC"
- board text added: "9"
- board text added: "CH343"
- board text added: "Cellar Door"
- board text added: "ESP32 4MB Flash CH343 USB/Serial"
- board text added: "G"
- board text added: "GND"
- board text added: "I2C SDA:14 SCL:13"
- board text added: "ICS-43434 I2S Mic SD:25 CK:26 WS:33"
- board text added: "IR Remote: 32"
- board text added: "JST SH: 27"
- board text added: "LED: 4"
- board text added: "NeoPix: 2"
- board text added: "RX"
- board text added: "TX"
- board text added: "USB PD Type C"
- board text added: "V+"
- board text removed: "S1"
- board text removed: "S2"
- board text removed: "S3"
