File: Adafruit Sparkle Motion WLED Friend.sch (EAGLE design)
At the start: 66 parts, among them IC1 CH343P, IC2 ICS-43434, IC4 74LVC2G34GW, IC5 74LVC2G34GW, Q1 AONR21307, Q5 DUAL NPN, SW1 KMR2, SW2 KMR2, SW3 SWITCH_SP3T_SMD_MSK13C01, U2 NCP718ASN500T1G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

Commit message: shop image & final board silk
Parts:
- added TP3, TP4: (no value), microbuilder:TESTPOINTROUND1.5MM
- R12: value 47K -> 10K
Connections:
- net !RESET: now also TP3.P$1
- net GPIO0: now also TP4.P$1
Other:
- note added: "2x3 GPIO"
- note added: "5V Level Shifter"
- note added: "I2S Microphone"
- note added: "Infrared Remote"
- note added: "JST SH"
- note added: "Outputs"
- note added: "Stemma QT I2C"
- moved on the sheet: C1, C11, C12, C13, C14, C15, C4, C9, CONN1G$1, D3, IC1, IC2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
